Commit message: fix(model): emit package:// mesh URIs in the generated URDF
- replace file:// URIs built from the generator's absolute working directory with package://humanoid_bringup/ plus the repo-relative assets path, which humanoid_bringup already installs
- remove the dependency of robot.urdf on the checkout location (/ws in the container, a home directory elsewhere) so regenerate-and-diff no longer depends on where it runs
- let Foxglove load the meshes, because it fetches only package:// URIs over the bridge and reads file:// from the viewer's own disk, which left the robot invisible
- regenerate robot.urdf; the only change is the mesh URI prefix, and robot.mjcf and safety_manifest.yaml are unchanged

File: model/generated/robot.urdf (robot description, URDF)
Before this commit: robot unitree_g1, 30 links, 29 joints
Links:
- link left_ankle_pitch_link: geometry collision mesh filename=package://humanoid_bringup/model/source/menagerie/unitree_g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; visual mesh filename=package://humanoid_bringup/model/source/menagerie/unitree_g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
- link left_ankle_roll_link: geometry collision mesh filename=package://humanoid_bringup/model/source/menagerie/unitree_g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; collision sphere radius=0.005
- link left_elbow_link: geometry collision mesh filename=package://humanoid_bringup/model/source/menagerie/unitree_g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; visual mesh filename=package://humanoid_bringup/model/source/menagerie/unitree_g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
- link left_hip_pitch_link: geometry collision mesh filename=package://humanoid_bringup/model/source/menagerie/unitree_g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; visual mesh filename=package://humanoid_bringup/model/source/menagerie/unitree_g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
- link left_hip_roll_link: geometry collision mesh filename=package://humanoid_bringup/model/source/menagerie/unitree_g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; visual mesh filename=package://humanoid_bringup/model/source/menagerie/unitree_g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
- link left_hip_yaw_link: geometry collision mesh filename=package://humanoid_bringup/model/source/menagerie/unitree_g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; visual mesh filename=package://humanoid_bringup/model/source/menagerie/unitree_g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
- link left_knee_link: geometry collision mesh filename=package://humanoid_bringup/model/source/menagerie/unitree_g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; visual mesh filename=package://humanoid_bringup/model/source/menagerie/unitree_g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
- link left_shoulder_pitch_link: geometry collision cylinder length=0.05 radius=0.03; collision mesh filename=package://humanoid_bringup/model/source/menagerie/unitree_g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
- link left_shoulder_roll_link: geometry collision cylinder length=0.03 radius=0.03; collision mesh filename=package://humanoid_bringup/model/source/menagerie/unitree_g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
- link left_shoulder_yaw_link: geometry collision mesh filename=package://humanoid_bringup/model/source/menagerie/unitree_g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; visual mesh filename=package://humanoid_bringup/model/source/menagerie/unitree_g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
- link left_wrist_pitch_link: geometry collision mesh filename=package://humanoid_bringup/model/source/menagerie/unitree_g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; visual mesh filename=package://humanoid_bringup/model/source/menagerie/unitree_g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
- link left_wrist_roll_link: geometry collision mesh filename=package://humanoid_bringup/model/source/menagerie/unitree_g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; visual mesh filename=package://humanoid_bringup/model/source/menagerie/unitree_g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
- link left_wrist_yaw_link: geometry collision mesh filename=package://humanoid_bringup/model/source/menagerie/unitree_g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; visual mesh filename=package://humanoid_bringup/model/source/menagerie/unitree_g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
- link pelvis: geometry collision mesh filename=package://humanoid_bringup/model/source/menagerie/unitree_g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; visual mesh filename=package://humanoid_bringup/model/source/menagerie/unitree_g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
- link right_ankle_pitch_link: geometry collision mesh filename=package://humanoid_bringup/model/source/menagerie/unitree_g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; visual mesh filename=package://humanoid_bringup/model/source/menagerie/unitree_g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
- link right_ankle_roll_link: geometry collision mesh filename=package://humanoid_bringup/model/source/menagerie/unitree_g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; collision sphere radius=0.005
- link right_elbow_link: geometry collision mesh filename=package://humanoid_bringup/model/source/menagerie/unitree_g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; visual mesh filename=package://humanoid_bringup/model/source/menagerie/unitree_g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
- link right_hip_pitch_link: geometry collision mesh filename=package://humanoid_bringup/model/source/menagerie/unitree_g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; visual mesh filename=package://humanoid_bringup/model/source/menagerie/unitree_g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
- link right_hip_roll_link: geometry collision mesh filename=package://humanoid_bringup/model/source/menagerie/unitree_g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; visual mesh filename=package://humanoid_bringup/model/source/menagerie/unitree_g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
- link right_hip_yaw_link: geometry collision mesh filename=package://humanoid_bringup/model/source/menagerie/unitree_g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; visual mesh filename=package://humanoid_bringup/model/source/menagerie/unitree_g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
- link right_knee_link: geometry collision mesh filename=package://humanoid_bringup/model/source/menagerie/unitree_g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; visual mesh filename=package://humanoid_bringup/model/source/menagerie/unitree_g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
- link right_shoulder_pitch_link: geometry collision cylinder length=0.05 radius=0.03; collision mesh filename=package://humanoid_bringup/model/source/menagerie/unitree_g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
- link right_shoulder_roll_link: geometry collision cylinder length=0.03 radius=0.03; collision mesh filename=package://humanoid_bringup/model/source/menagerie/unitree_g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
- link right_shoulder_yaw_link: geometry collision mesh filename=package://humanoid_bringup/model/source/menagerie/unitree_g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; visual mesh filename=package://humanoid_bringup/model/source/menagerie/unitree_g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
- link right_wrist_pitch_link: geometry collision mesh filename=package://humanoid_bringup/model/source/menagerie/unitree_g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; visual mesh filename=package://humanoid_bringup/model/source/menagerie/unitree_g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
- link right_wrist_roll_link: geometry collision mesh filename=package://humanoid_bringup/model/source/menagerie/unitree_g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; visual mesh filename=package://humanoid_bringup/model/source/menagerie/unitree_g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
- link right_wrist_yaw_link: geometry collision mesh filename=package://humanoid_bringup/model/source/menagerie/unitree_g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; visual mesh filename=package://humanoid_bringup/model/source/menagerie/unitree_g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
- link torso_link: geometry collision mesh filename=package://humanoid_bringup/model/source/menagerie/unitree_g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; visual mesh filename=package://humanoid_bringup/model/source/menagerie/unitree_g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
- link waist_roll_link: geometry collision mesh filename=package://humanoid_bringup/model/source/menagerie/unitree_g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; visual mesh filename=package://humanoid_bringup/model/source/menagerie/unitree_g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
- link waist_yaw_link: geometry collision mesh filename=package://humanoid_bringup/model/source/menagerie/unitree_g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; visual mesh filename=package://humanoid_bringup/model/source/menagerie/unitree_g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

Commit message: feat(model): emit the pelvis imu from the ingested model
- ingest the imu site named by `imu_site` in ingest.yaml into an optional `imu` block of robot_model.yaml
- add the `imu` block to the schema and check its link and quaternion in validate.py
- emit an MJCF site with one framequat, gyro and accelerometer, a URDF imu_link frame, and a ros2_control sensor with the ten imu_sensor_broadcaster interfaces
- fix the generated MJCF dropping the menagerie imu sensors, which left simulation with no inertial feedback

File: model/generated/robot.urdf (robot description, URDF)
Before this commit: robot unitree_g1, 30 links, 29 joints
Links:
- added link imu_link
Joints:
- added joint imu_joint: type fixed, parent pelvis, child imu_link, origin xyz=0.04525 0 -0.08339 rpy=0 0 0
