Commit message: refactor(model): lay out unitree_g1 like every other robot
- move G1's source (robot_model.yaml, contact overlay, import config, vendored Menagerie) to model/robots/unitree_g1/source/ and its outputs to model/robots/unitree_g1/generated/, matching the benches
- compute the MJCF meshdir from the robot's own generated/ directory instead of a hard-coded "model/generated", which any second MJCF robot would have got wrong
- repoint the bringup install rules, the SIL launch defaults, the actuator-system and MuJoCo test paths, the CI variable, and the docs
- cover every robot's generated/ in CODEOWNERS, so the benches' safety manifests and firmware configs get the same review as G1's
- leave robot.mjcf and safety_manifest.yaml byte-identical; robot.urdf changes only its package:// mesh URIs

File: model/robots/unitree_g1/generated/robot.urdf (robot description, URDF)
Before this commit: robot unitree_g1, 31 links, 30 joints
Links:
- link left_ankle_pitch_link: geometry collision mesh filename=package://humanoid_bringup/model/robots/unitree_g1/source/m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; visual mesh filename=package://humanoid_bringup/model/robots/unitree_g1/source/m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
- link left_ankle_roll_link: geometry collision mesh filename=package://humanoid_bringup/model/robots/unitree_g1/source/m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; collision sphere radius=0.005
- link left_elbow_link: geometry collision mesh filename=package://humanoid_bringup/model/robots/unitree_g1/source/m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; visual mesh filename=package://humanoid_bringup/model/robots/unitree_g1/source/m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
- link left_hip_pitch_link: geometry collision mesh filename=package://humanoid_bringup/model/robots/unitree_g1/source/m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; visual mesh filename=package://humanoid_bringup/model/robots/unitree_g1/source/m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
- link left_hip_roll_link: geometry collision mesh filename=package://humanoid_bringup/model/robots/unitree_g1/source/m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; visual mesh filename=package://humanoid_bringup/model/robots/unitree_g1/source/m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
- link left_hip_yaw_link: geometry collision mesh filename=package://humanoid_bringup/model/robots/unitree_g1/source/m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; visual mesh filename=package://humanoid_bringup/model/robots/unitree_g1/source/m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
- link left_knee_link: geometry collision mesh filename=package://humanoid_bringup/model/robots/unitree_g1/source/m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; visual mesh filename=package://humanoid_bringup/model/robots/unitree_g1/source/m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
- link left_shoulder_pitch_link: geometry collision cylinder length=0.05 radius=0.03; collision mesh filename=package://humanoid_bringup/model/robots/unitree_g1/source/m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
- link left_shoulder_roll_link: geometry collision cylinder length=0.03 radius=0.03; collision mesh filename=package://humanoid_bringup/model/robots/unitree_g1/source/m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
- link left_shoulder_yaw_link: geometry collision mesh filename=package://humanoid_bringup/model/robots/unitree_g1/source/m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; visual mesh filename=package://humanoid_bringup/model/robots/unitree_g1/source/m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
- link left_wrist_pitch_link: geometry collision mesh filename=package://humanoid_bringup/model/robots/unitree_g1/source/m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; visual mesh filename=package://humanoid_bringup/model/robots/unitree_g1/source/m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
- link left_wrist_roll_link: geometry collision mesh filename=package://humanoid_bringup/model/robots/unitree_g1/source/m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; visual mesh filename=package://humanoid_bringup/model/robots/unitree_g1/source/m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
- link left_wrist_yaw_link: geometry collision mesh filename=package://humanoid_bringup/model/robots/unitree_g1/source/m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; visual mesh filename=package://humanoid_bringup/model/robots/unitree_g1/source/m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
- link pelvis: geometry collision mesh filename=package://humanoid_bringup/model/robots/unitree_g1/source/m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; visual mesh filename=package://humanoid_bringup/model/robots/unitree_g1/source/m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
- link right_ankle_pitch_link: geometry collision mesh filename=package://humanoid_bringup/model/robots/unitree_g1/source/m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; visual mesh filename=package://humanoid_bringup/model/robots/unitree_g1/source/m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
- link right_ankle_roll_link: geometry collision mesh filename=package://humanoid_bringup/model/robots/unitree_g1/source/m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; collision sphere radius=0.005
- link right_elbow_link: geometry collision mesh filename=package://humanoid_bringup/model/robots/unitree_g1/source/m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; visual mesh filename=package://humanoid_bringup/model/robots/unitree_g1/source/m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
- link right_hip_pitch_link: geometry collision mesh filename=package://humanoid_bringup/model/robots/unitree_g1/source/m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; visual mesh filename=package://humanoid_bringup/model/robots/unitree_g1/source/m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
- link right_hip_roll_link: geometry collision mesh filename=package://humanoid_bringup/model/robots/unitree_g1/source/m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; visual mesh filename=package://humanoid_bringup/model/robots/unitree_g1/source/m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
- link right_hip_yaw_link: geometry collision mesh filename=package://humanoid_bringup/model/robots/unitree_g1/source/m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; visual mesh filename=package://humanoid_bringup/model/robots/unitree_g1/source/m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
- link right_knee_link: geometry collision mesh filename=package://humanoid_bringup/model/robots/unitree_g1/source/m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; visual mesh filename=package://humanoid_bringup/model/robots/unitree_g1/source/m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
- link right_shoulder_pitch_link: geometry collision cylinder length=0.05 radius=0.03; collision mesh filename=package://humanoid_bringup/model/robots/unitree_g1/source/m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
- link right_shoulder_roll_link: geometry collision cylinder length=0.03 radius=0.03; collision mesh filename=package://humanoid_bringup/model/robots/unitree_g1/source/m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
- link right_shoulder_yaw_link: geometry collision mesh filename=package://humanoid_bringup/model/robots/unitree_g1/source/m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; visual mesh filename=package://humanoid_bringup/model/robots/unitree_g1/source/m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
- link right_wrist_pitch_link: geometry collision mesh filename=package://humanoid_bringup/model/robots/unitree_g1/source/m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; visual mesh filename=package://humanoid_bringup/model/robots/unitree_g1/source/m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
- link right_wrist_roll_link: geometry collision mesh filename=package://humanoid_bringup/model/robots/unitree_g1/source/m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; visual mesh filename=package://humanoid_bringup/model/robots/unitree_g1/source/m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
- link right_wrist_yaw_link: geometry collision mesh filename=package://humanoid_bringup/model/robots/unitree_g1/source/m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; visual mesh filename=package://humanoid_bringup/model/robots/unitree_g1/source/m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
- link torso_link: geometry collision mesh filename=package://humanoid_bringup/model/robots/unitree_g1/source/m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; visual mesh filename=package://humanoid_bringup/model/robots/unitree_g1/source/m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
- link waist_roll_link: geometry collision mesh filename=package://humanoid_bringup/model/robots/unitree_g1/source/m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; visual mesh filename=package://humanoid_bringup/model/robots/unitree_g1/source/m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
- link waist_yaw_link: geometry collision mesh filename=package://humanoid_bringup/model/robots/unitree_g1/source/m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; visual mesh filename=package://humanoid_bringup/model/robots/unitree_g1/source/m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
